Commit message: ”首次提交“

File: ws02_tools/install/cpp7_gazebo/share/cpp7_gazebo/urdf/xacro/car_laser.urdf.xacro (robot description, xacro)
@@ -3,5 +3,5 @@
     <!-- 1.声明参数 -->
     <xacro:property name="laser_radius" value="0.08"/>
-    <xacro:property name="laser_length" value="0.08"/>
+    <xacro:property name="laser_length" value="0.10"/>
     <xacro:property name="laser_mass" value="1.76"/>
     <!-- 关节偏移量 -->

File: ws02_tools/install/cpp7_gazebo/share/cpp7_gazebo/urdf/xacro/car_urdf.xacro (robot description, xacro)
@@ -6,5 +6,12 @@
    <xacro:include filename="car_camera.urdf.xacro"/>
    <xacro:include filename="car_laser.urdf.xacro"/>
+   <xacro:include filename="car_kinect.urdf.xacro"/>
    <!-- 运动控制 -->
-   <xacro:include filename="../gazebo/car_move.urdf.xacro"/>
+   <xacro:include filename="../gazebo/move.xacro"/>
+   <!-- 雷达 -->
+   <xacro:include filename="../gazebo/laser.xacro"/>
+   <!-- 摄像头 -->
+   <xacro:include filename="../gazebo/camera.xacro"/>
+   <!-- 深度摄像头 -->
+   <xacro:include filename="../gazebo/kinect.xacro"/>
  </robot>
